File: hw/controller/SuperClockController.kicad_pcb (KiCad board)
At the start: 2 copper layers, 139.7 x 48.3 mm, 82 parts, among them J1 Led Cathodes, J2 Led Anodes, J3 Yellow LED 0, J4 Yellow LED 1, J5 USB_A, J6 ATmega ISP, Q1 AO3416A, Q10 AO3416A, Q11 AO3416A, Q12 AO3416A, Q13 AO3416A, Q14 AO3416A, Q15 AO3416A, Q16 AO3416A, Q17 AO3416A, Q18 AO3416A, Q2 AO3416A, Q3 AO3416A, Q4 AO3416A, Q5 AO3416A, Q6 AO3416A, Q7 AO3416A, Q8 AO3416A, Q9 AO3416A, SW1 SW_Push, SW2 SW_Push, SW3 SW_Push, U1 ATmega32A-A, U2 DS3231SN, U3 DS1307ZN, Y1 16MHz, Y2 32.768kHz

Commit message: Mark R1-R17 as DNP, replace AO3416 with 2N7002K and update docs.
It turned out that green LEDs do not like the reverse voltage at all, and they started slowly failing in a few months. So let's combat LED ghosting by using MOSFETs with lower parasitic capacitance instead of adding pull-up resistors.
Parts:
- Q1, Q10, Q11, Q12, Q13, Q14, Q15, Q16, Q17, Q18, Q2, Q3, Q4, Q5, Q6, Q7, Q8, Q9: value AO3416A -> 2N7002K
- R1, R10, R11, R12, R13, R14, R15, R16, R17, R2, R3, R4, R5, R6, R7, R8, R9: value 220 -> ~
