File: hw/controller/SuperClockController.kicad_sch (KiCad schematic)
At the start: 82 parts, among them J1 Led Cathodes, J2 Led Anodes, J3 Yellow LED 0, J4 Yellow LED 1, J5 USB_A, J6 ATmega ISP, Q1 IRLML2502, Q10 IRLML2502, Q11 IRLML2502, Q12 IRLML2502, Q13 IRLML2502, Q14 IRLML2502, Q15 IRLML2502, Q16 IRLML2502, Q17 IRLML2502, Q18 IRLML2502, Q2 IRLML2502, Q3 IRLML2502, Q4 IRLML2502, Q5 IRLML2502, Q6 IRLML2502, Q7 IRLML2502, Q8 IRLML2502, Q9 IRLML2502, SW1 SW_Push, SW2 SW_Push, SW3 SW_Push, U1 ATmega32A-A, U2 DS3231SN, U3 DS1307ZN, Y1 16MHz, Y2 32.768kHz

Commit message: Replace IRLML2505 to AO3416A
This one claims to have ESD-protected gates, should be easier to handle
Parts:
- Q1, Q10, Q11, Q12, Q13, Q14, Q15, Q16, Q17, Q18, Q2, Q3, Q4, Q5, Q6, Q7, Q8, Q9: value IRLML2502 -> AO3416A
Changed lines of the file:
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@@
 			)
 		)
-		(property "Value" "IRLML2502"
+		(property "Value" "AO3416A"
 			(at 271.78 251.4599 0)
 			(effects
@@
 			)
 		)
-		(property "Value" "IRLML2502"
+		(property "Value" "AO3416A"
 			(at 271.78 120.6499 0)
 			(effects
@@
 			)
 		)
-		(property "Value" "IRLML2502"
+		(property "Value" "AO3416A"
 			(at 271.78 93.9799 0)
 			(effects
@@
 			)
 		)
-		(property "Value" "IRLML2502"
+		(property "Value" "AO3416A"
 			(at 309.88 147.3199 0)
 			(effects
@@
 			)
 		)
-		(property "Value" "IRLML2502"
+		(property "Value" "AO3416A"
 			(at 309.88 95.2499 0)
 			(effects
@@
 			)
 		)
-		(property "Value" "IRLML2502"
+		(property "Value" "AO3416A"
 			(at 309.88 173.9899 0)
 			(effects
@@
 			)
 		)
-		(property "Value" "IRLML2502"
+		(property "Value" "AO3416A"
 			(at 309.88 121.9199 0)
 			(effects
@@
 			)
 		)
-		(property "Value" "IRLML2502"
+		(property "Value" "AO3416A"
 			(at 271.78 199.3899 0)
 			(effects
@@
 			)
 		)
-		(property "Value" "IRLML2502"
+		(property "Value" "AO3416A"
 			(at 309.88 41.9099 0)
 			(effects
@@
 			)
 		)
-		(property "Value" "IRLML2502"
+		(property "Value" "AO3416A"
 			(at 55.88 173.9899 0)
 			(effects
@@
 			)
 		)
-		(property "Value" "IRLML2502"
+		(property "Value" "AO3416A"
 			(at 271.78 40.6399 0)
 			(effects
@@
 			)
 		)
-		(property "Value" "IRLML2502"
+		(property "Value" "AO3416A"
 			(at 271.78 224.7899 0)
 			(effects
@@
 			)
 		)
-		(property "Value" "IRLML2502"
+		(property "Value" "AO3416A"
 			(at 271.78 172.7199 0)
 			(effects
@@
 			)
 		)
-		(property "Value" "IRLML2502"
+		(property "Value" "AO3416A"
 			(at 271.78 146.0499 0)
 			(effects
@@
 			)
 		)
-		(property "Value" "IRLML2502"
+		(property "Value" "AO3416A"
 			(at 309.88 68.5799 0)
 			(effects
@@
 			)
 		)
-		(property "Value" "IRLML2502"
+		(property "Value" "AO3416A"
 			(at 271.78 67.3099 0)
 			(effects
@@
 			)
 		)
-		(property "Value" "IRLML2502"
+		(property "Value" "AO3416A"
 			(at 309.88 226.0599 0)
 			(effects
@@
 			)
 		)
-		(property "Value" "IRLML2502"
+		(property "Value" "AO3416A"
 			(at 309.88 200.6599 0)
 			(effects

Commit message: Mark R1-R17 as DNP, replace AO3416 with 2N7002K and update docs.
It turned out that green LEDs do not like the reverse voltage at all, and they started slowly failing in a few months. So let's combat LED ghosting by using MOSFETs with lower parasitic capacitance instead of adding pull-up resistors.
Parts:
- Q1, Q10, Q11, Q12, Q13, Q14, Q15, Q16, Q17, Q18, Q2, Q3, Q4, Q5, Q6, Q7, Q8, Q9: value AO3416A -> 2N7002K
- R1, R10, R11, R12, R13, R14, R15, R16, R17, R2, R3, R4, R5, R6, R7, R8, R9: value 220 -> (none); now not fitted
